File: Hardware/Ares-01/Ares-01.kicad_pcb (KiCad board)
At the start: 2 copper layers, 81.5 x 87.2 mm, 26 parts, among them J1 BTS7960, J12 XT30, J13 TCRT5000_1, J14 TCRT5000_2, J15 TCRT5000_3, J2 BTS7960, J3 Sharp, J4 Sharp, J5 Sharp, J6 Sharp, J7 Sharp, J8 Qtr8a, J9 Ssd1306 Arduino Pic, SW1 Switch, SW2 SW_Push, SW3 SW_Push, U1 L7805, U2 AMS1117, U3 CD74HC4067M

Commit message: Se actualizo PCB
Parts:
- removed J8: Qtr8a, Connector_JST:JST_XH_B10B-XH-A_1x10_P2.50mm_Vertical
- added J10: Conn_01x10_Pin, Connector_JST:JST_XH_B10B-XH-A_1x10_P2.50mm_Vertical, F.Cu at (223.8, 66.2)
Connections:
- U3 pad 2: D8 -> D1
- U3 pad 3: D7 -> D2
- U3 pad 4: D6 -> D3
- U3 pad 5: D5 -> D4
- U3 pad 6: D4 -> D5
- U3 pad 7: D3 -> D6
- U3 pad 8: D2 -> D7
- U3 pad 9: D1 -> D8
Routing:
- net COM: track 9.57 -> 45.7 mm
- net 3.3V: track 191.5 -> 208.8 mm
- net VCC: track 115.5 -> 119.9 mm
- net SCL: track 27.6 -> 26.3 mm
- net D5: track 5.56 -> 6.43 mm
- net D4: track 5.54 -> 6.41 mm
- net D8: track 5.61 -> 6.48 mm
- net D7: track 5.59 -> 6.46 mm
- net D6: track 5.57 -> 6.45 mm
- net D3: track 5.56 -> 6.40 mm
- net D2: track 5.57 -> 6.38 mm
- net D1: track 5.59 -> 6.36 mm
